Commit message: Working on Camera Sensor

File: arduinobot_description/urdf/camera.xacro (robot description, xacro)
@@ -8,6 +8,7 @@
                     scale="0.01 0.01 0.01" />
             </geometry>
+            <material name="red" />
         </visual>
-        <collison>
+        <collision>
             <origin xyz="-0.1 0.13 0.14" rpy="-${pi / 2.0} 0 -${pi / 2.0}" />
             <geometry>
@@ -15,5 +16,5 @@
                     scale="0.01 0.01 0.01" />
             </geometry>
-        </collison>
+        </collision>
         <xacro:default_inertia mass="0.001" />
     </link>
@@ -23,31 +24,24 @@
         <child link="rgb_camera" />
     </joint>
-    <!-- <gazebo reference="camera_link">
-        <material>Gazebo/Red</material>
+    <gazebo reference="camera_link">
         <sensor name="camera_sensor" type="camera">
-            <pose>0 0 0 0 0 0</pose>
+            <camera name="camera">
+                <camera_info_topic>camera_info</camera_info_topic>
+                <horizontal_fov>1.15</horizontal_fov>
+                <image>
+                    <width>2304</width>
+                    <height>1296</height>
+                </image>
+                <clip>
+                    <near>0.1</near>
+                    <far>100</far>
+                </clip>
+            </camera>
+            <always_on>1</always_on>
+            <update_rate>30</update_rate>
             <visualize>true</visualize>
-            <update_rate>10.0</update_rate>
-            <plugin name="camera_controller" filename="libgazebo_ros_camera.so">
-                <frame_name>camera_link</frame_name>
-            </plugin>
+            <topic>image_raw</topic>
+            <frame_id>rgb_camera</frame_id>
         </sensor>
-    </gazebo> -->
-    <sensor name="camera" type="camera">
-        <camera>
-            <horizontal_fov>1.047</horizontal_fov>
-            <image>
-                <width>320</width>
-                <height>240</height>
-            </image>
-            <clip>
-                <near>0.1</near>
-                <far>100</far>
-            </clip>
-        </camera>
-        <always_on>1</always_on>
-        <update_rate>30</update_rate>
-        <visualize>true</visualize>
-        <topic>camera</topic>
-    </sensor>
+    </gazebo>
 </robot>

File: arduinobot_description/urdf/common_properties.xacro (robot description, xacro)
@@ -9,4 +9,7 @@
     <material name="green">
         <color rgba="0 0.5 0 1" />
+    </material>
+    <material name="red">
+        <color rgba="1 0 0 1" />
     </material>
     <material name="orange">

Commit message: working camera sensor

File: arduinobot_description/urdf/camera.xacro (robot description, xacro)
@@ -1,5 +1,5 @@
 <?xml version="1.0"?>
 <robot xmlns:xacro="http://www.ros.org/wiki/xacro">
-    <link name="rgb_camera">
+    <link name="rgb_camera_link">
         <visual>
             <origin xyz="-0.1 0.13 0.14" rpy="-${pi / 2.0} 0 -${pi / 2.0}" />
@@ -22,10 +22,10 @@
         <origin xyz="0 0.45 0.2" rpy="0 -0.5 1.57" />
         <parent link="base_link" />
-        <child link="rgb_camera" />
+        <child link="rgb_camera_link" />
     </joint>
-    <gazebo reference="camera_link">
+    <gazebo reference="rgb_camera_link">
         <sensor name="camera_sensor" type="camera">
             <camera name="camera">
-                <camera_info_topic>camera_info</camera_info_topic>
+                <camera_info_topic>rgb_camera/camera_info</camera_info_topic>
                 <horizontal_fov>1.15</horizontal_fov>
                 <image>
@@ -41,7 +41,18 @@
             <update_rate>30</update_rate>
             <visualize>true</visualize>
-            <topic>image_raw</topic>
-            <frame_id>rgb_camera</frame_id>
+            <topic>rgb_camera/image_raw</topic>
         </sensor>
     </gazebo>
+    <gazebo>
+        <plugin
+            filename="gz-sim-joint-state-publisher-system"
+            name="gz::sim::systems::JointStatePublisher">
+            <topic>joint_states</topic>
+            <joint_name>joint_1</joint_name>
+            <joint_name>joint_2</joint_name>
+            <joint_name>joint_3</joint_name>
+            <joint_name>joint_4</joint_name>
+            <joint_name>joint_5</joint_name>
+        </plugin>
+    </gazebo>
 </robot>
