Commit message: moveit integration

File: arduinobot_description/urdf/arduinobot.urdf.xacro (robot description, xacro)
@@ -2,4 +2,6 @@
 <robot name="arduinobot" xmlns:xacro="http://www.ros.org/wiki/xacro">
     <xacro:include filename="common_properties.xacro" />
+    <xacro:include filename="arduinobot_gazebo.xacro"/>
+    <xacro:include filename="arduinobot_control.xacro"/>
     <xacro:include filename="robot_structure.xacro" />
     <xacro:include filename="camera.xacro" />

File: arduinobot_description/urdf/camera.xacro (robot description, xacro)
@@ -44,15 +44,3 @@
         </sensor>
     </gazebo>
-    <gazebo>
-        <plugin
-            filename="gz-sim-joint-state-publisher-system"
-            name="gz::sim::systems::JointStatePublisher">
-            <topic>joint_states</topic>
-            <joint_name>joint_1</joint_name>
-            <joint_name>joint_2</joint_name>
-            <joint_name>joint_3</joint_name>
-            <joint_name>joint_4</joint_name>
-            <joint_name>joint_5</joint_name>
-        </plugin>
-    </gazebo>
 </robot>

File: arduinobot_description/urdf/robot_structure.xacro (robot description, xacro)
@@ -66,5 +66,5 @@
         <xacro:default_inertia mass="0.1" />
     </link>
-    <link name="horrizontal_arm">
+    <link name="horizontal_arm">
         <visual>
             <origin xyz="-0.03 -0.4 -0.06" rpy="${pi / 2.0} 0 ${pi / 2.0}" />
@@ -162,11 +162,11 @@
         <origin xyz="0 0 0.8" rpy="0 0 0" />
         <parent link="forward_drive_arm" />
-        <child link="horrizontal_arm" />
+        <child link="horizontal_arm" />
         <axis xyz="1 0 0" />
         <limit lower="-${pi / 2.0}" upper="${pi / 2.0}" effort="${effort}" velocity="${velocity}" />
     </joint>
-    <joint name="horrizontal_arm_to_claw_support" type="fixed">
+    <joint name="horizontal_arm_to_claw_support" type="fixed">
         <origin xyz="0 0.82 0" rpy="0 0 0" />
-        <parent link="horrizontal_arm" />
+        <parent link="horizontal_arm" />
         <child link="claw_support" />
     </joint>

Commit message: learning

File: arduinobot_description/urdf/arduinobot.urdf.xacro (robot description, xacro)
@@ -1,4 +1,5 @@
 <?xml version="1.0"?>
 <robot name="arduinobot" xmlns:xacro="http://www.ros.org/wiki/xacro">
+    <xacro:arg name="is_sim" default="true"/>
     <xacro:include filename="common_properties.xacro" />
     <xacro:include filename="arduinobot_gazebo.xacro"/>

File: arduinobot_description/urdf/arduinobot_control.xacro (robot description, xacro)
@@ -2,7 +2,20 @@
 <robot xmlns:xacro="http://www.ros.org/wiki/xacro">
     <ros2_control type="system" name="RobotSystem">
-            <hardware>
-                <plugin>gz_ros2_control/GazeboSimSystem</plugin>
-            </hardware>
+            <!-- ros2 control Gazebo-->
+            <xacro:if value="$(arg is_sim)">
+                <hardware>
+                    <plugin>gz_ros2_control/GazeboSimSystem</plugin>
+                </hardware>
+                <joint name="joint_5">
+                <param name="mimic">joint_4</param>
+                <param name="multiplier">-1</param>
+            </joint>
+            </xacro:if>
+            <xacro:unless value="$(arg is_sim)">
+                <hardware>
+                    <plugin>arduinobot_controller/ArduinobotInterface</plugin>
+                    <param name="port">/dev/ttyUSB0</param>
+                </hardware>
+            </xacro:unless>
             <joint name="joint_1">
                 <command_interface name="position">
@@ -33,8 +46,4 @@
                 <state_interface name="position"/>
             </joint>
-            <joint name="joint_5">
-                <param name="mimic">joint_4</param>
-                <param name="multiplier">-1</param>
-            </joint>
     </ros2_control>
 </robot>

File: arduinobot_description/urdf/robot_structure.xacro (robot description, xacro)
@@ -57,5 +57,5 @@
             <material name="grey" />
         </visual>
-        <collison>
+        <collision>
             <origin xyz="0.19 0.06 -0.08" rpy="0 -${pi / 2.0} ${pi / 2.0}" />
             <geometry>
@@ -63,5 +63,5 @@
                     scale="0.01 0.01 0.01" />
             </geometry>
-        </collison>
+        </collision>
         <xacro:default_inertia mass="0.1" />
     </link>
@@ -76,5 +76,5 @@
             <material name="grey" />
         </visual>
-        <collison>
+        <collision>
             <origin xyz="-0.03 -0.4 -0.06" rpy="${pi / 2.0} 0 ${pi / 2.0}" />
             <geometry>
@@ -83,5 +83,5 @@
                 <material name="grey" />
             </geometry>
-        </collison>
+        </collision>
         <xacro:default_inertia mass="0.1" />
     </link>
@@ -95,5 +95,5 @@
             <material name="yellow" />
         </visual>
-        <collison>
+        <collision>
             <origin xyz="0 -0.05 -0.15" rpy="0 0 ${pi / 2.0}" />
             <geometry>
@@ -101,5 +101,5 @@
                     scale="0.01 0.01 0.01" />
             </geometry>
-        </collison>
+        </collision>
         <xacro:default_inertia mass="0.05" />
     </link>
@@ -113,5 +113,5 @@
             <material name="green" />
         </visual>
-        <collison>
+        <collision>
             <origin xyz="-0.1 0.5 -0.1" rpy="0 0 -${pi / 2.0}" />
             <geometry>
@@ -119,5 +119,5 @@
                     scale="0.01 0.01 0.01" />
             </geometry>
-        </collison>
+        </collision>
         <xacro:default_inertia mass="0.01" />
     </link>
@@ -140,5 +140,5 @@
         <xacro:default_inertia mass="0.01" />
     </link>
-    <joint name="world_base_link_joint" type="fixed">
+    <joint name="virtual_joint" type="fixed">
         <origin xyz="0 0 0" rpy="0 0 0" />
         <parent link="world" />
