Commit message: completed tutorial

File: arduinobot_description/urdf/arduinobot_control.xacro (robot description, xacro)
@@ -1,6 +1,5 @@
 <?xml version="1.0"?>
 <robot xmlns:xacro="http://www.ros.org/wiki/xacro">
-    <ros2_control type="system" name="RobotSystem">
-            <!-- ros2 control Gazebo-->
+    <ros2_control name="RobotSystem" type="system" >
             <xacro:if value="$(arg is_sim)">
                 <hardware>
@@ -8,7 +7,7 @@
                 </hardware>
                 <joint name="joint_5">
-                <param name="mimic">joint_4</param>
-                <param name="multiplier">-1</param>
-            </joint>
+                    <param name="mimic">joint_4</param>
+                    <param name="multiplier">-1</param>
+                </joint>
             </xacro:if>
             <xacro:unless value="$(arg is_sim)">
@@ -42,5 +41,5 @@
                 <command_interface name="position">
                     <param name="min">-${pi / 2.0}</param>
-                    <param name="max">0.0</param>
+                    <param name="max">0.00001</param>
                 </command_interface>
                 <state_interface name="position"/>

File: arduinobot_description/urdf/arduinobot_gazebo.xacro (robot description, xacro)
@@ -1,6 +1,5 @@
 <?xml version="1.0"?>
 <robot xmlns:xacro="http://www.ros.org/wiki/xacro">
-<!--
-    <gazebo>
+    <!-- <gazebo>
         <plugin
             filename="gz-sim-joint-state-publisher-system"
@@ -14,9 +13,40 @@
         </plugin>
     </gazebo>
-     -->
     <gazebo>
         <plugin
-            filename="gz_ros2_control-system"
-            name="gz_ros2_control::GazeboSimROS2ControlPlugin">
+            filename="gz-sim-joint-position-controller-system"
+            name="gz::sim::systems::JointPositionController">
+            <joint_name>joint_1</joint_name>
+            <p_gain>1</p_gain>
+            <i_gain>0.1</i_gain>
+            <d_gain>0.01</d_gain>
+        </plugin>
+        <plugin
+            filename="gz-sim-joint-position-controller-system"
+            name="gz::sim::systems::JointPositionController">
+            <joint_name>joint_2</joint_name>
+            <p_gain>1</p_gain>
+            <i_gain>0.1</i_gain>
+            <d_gain>0.01</d_gain>
+        </plugin>
+        <plugin
+            filename="gz-sim-joint-position-controller-system"
+            name="gz::sim::systems::JointPositionController">
+            <joint_name>joint_3</joint_name>
+            <p_gain>1</p_gain>
+            <i_gain>0.1</i_gain>
+            <d_gain>0.01</d_gain>
+        </plugin>
+        <plugin
+            filename="gz-sim-joint-position-controller-system"
+            name="gz::sim::systems::JointPositionController">
+            <joint_name>joint_4</joint_name>
+            <p_gain>1</p_gain>
+            <i_gain>0.1</i_gain>
+            <d_gain>0.01</d_gain>
+        </plugin>
+    </gazebo> -->
+    <gazebo>
+        <plugin filename="gz_ros2_control-system" name="gz_ros2_control::GazeboSimROS2ControlPlugin">
             <parameters>$(find arduinobot_controller)/config/arduinobot_controllers.yaml</parameters>
         </plugin>

File: arduinobot_description/urdf/camera.xacro (robot description, xacro)
@@ -3,16 +3,16 @@
     <link name="rgb_camera_link">
         <visual>
-            <origin xyz="-0.1 0.13 0.14" rpy="-${pi / 2.0} 0 -${pi / 2.0}" />
+            <origin xyz="-0.01 0.013 0.014" rpy="-${pi / 2.0} 0 -${pi / 2.0}" />
             <geometry>
                 <mesh filename="package://arduinobot_description/meshes/pi_camera.STL"
-                    scale="0.01 0.01 0.01" />
+                    scale="0.001 0.001 0.001" />
             </geometry>
             <material name="red" />
         </visual>
         <collision>
-            <origin xyz="-0.1 0.13 0.14" rpy="-${pi / 2.0} 0 -${pi / 2.0}" />
+            <origin xyz="-0.01 0.013 0.014" rpy="-${pi / 2.0} 0 -${pi / 2.0}" />
             <geometry>
                 <mesh filename="package://arduinobot_description/meshes/pi_camera.STL"
-                    scale="0.01 0.01 0.01" />
+                    scale="0.001 0.001 0.001" />
             </geometry>
         </collision>
@@ -20,5 +20,5 @@
     </link>
     <joint name="rgb_camera_joint" type="fixed">
-        <origin xyz="0 0.45 0.2" rpy="0 -0.5 1.57" />
+        <origin xyz="0 0.045 0.02" rpy="0 -0.5 1.57" />
         <parent link="base_link" />
         <child link="rgb_camera_link" />

File: arduinobot_description/urdf/robot_structure.xacro (robot description, xacro)
@@ -6,7 +6,7 @@
         <inertial>
             <mass value="${mass}" />
-            <inertia ixx="1.0" ixy="0.0" ixz="0.0"
-                iyy="1.0" iyz="0.0"
-                izz="1.0" />
+            <inertia ixx="0.001" ixy="0.0" ixz="0.0"
+                iyy="0.001" iyz="0.0"
+                izz="0.001" />
         </inertial>
     </xacro:macro>
@@ -14,62 +14,62 @@
     <link name="base_link">
         <visual>
-            <origin xyz="-0.5 -0.5 0" rpy="0 0 0" />
+            <origin xyz="-0.05 -0.05 0" rpy="0 0 0" />
             <geometry>
                 <mesh filename="package://arduinobot_description/meshes/basement.STL"
-                    scale="0.01 0.01 0.01" />
+                    scale="0.001 0.001 0.001" />
             </geometry>
             <material name="blue" />
         </visual>
         <collision>
-            <origin xyz="-0.5 -0.5 0" rpy="0 0 0" />
+            <origin xyz="-0.05 -0.05 0" rpy="0 0 0" />
             <geometry>
                 <mesh filename="package://arduinobot_description/meshes/basement.STL"
-                    scale="0.01 0.01 0.01" />
+                    scale="0.001 0.001 0.001" />
             </geometry>
         </collision>
-        <xacro:default_inertia mass="1.0" />
+        <xacro:default_inertia mass="0.1" />
     </link>
     <link name="base_plate">
         <visual>
-            <origin xyz="-0.39 -0.39 -0.56" rpy="0 0 0" />
+            <origin xyz="-0.039 -0.039 -0.056" rpy="0 0 0" />
             <geometry>
                 <mesh filename="package://arduinobot_description/meshes/base_plate.STL"
-                    scale="0.01 0.01 0.01" />
+                    scale="0.001 0.001 0.001" />
             </geometry>
             <material name="orange" />
         </visual>
         <collision>
-            <origin xyz="-0.39 -0.39 -0.56" rpy="0 0 0" />
+            <origin xyz="-0.039 -0.039 -0.056" rpy="0 0 0" />
             <geometry>
                 <mesh filename="package://arduinobot_description/meshes/base_plate.STL"
-                    scale="0.01 0.01 0.01" />
+                    scale="0.001 0.001 0.001" />
             </geometry>
         </collision>
-        <xacro:default_inertia mass="0.1" />
+        <xacro:default_inertia mass="0.01" />
     </link>
     <link name="forward_drive_arm">
         <visual>
-            <origin xyz="0.19 0.06 -0.08" rpy="0 -${pi / 2.0} ${pi / 2.0}" />
+            <origin xyz="0.019 0.006 -0.008" rpy="0 -${pi / 2.0} ${pi / 2.0}" />
             <geometry>
                 <mesh filename="package://arduinobot_description/meshes/forward_drive_arm.STL"
-                    scale="0.01 0.01 0.01" />
+                    scale="0.001 0.001 0.001" />
             </geometry>
             <material name="grey" />
         </visual>
         <collision>
-            <origin xyz="0.19 0.06 -0.08" rpy="0 -${pi / 2.0} ${pi / 2.0}" />
+            <origin xyz="0.019 0.006 -0.008" rpy="0 -${pi / 2.0} ${pi / 2.0}" />
             <geometry>
                 <mesh filename="package://arduinobot_description/meshes/forward_drive_arm.STL"
-                    scale="0.01 0.01 0.01" />
+                    scale="0.001 0.001 0.001" />
             </geometry>
         </collision>
-        <xacro:default_inertia mass="0.1" />
+        <xacro:default_inertia mass="0.01" />
     </link>
     <link name="horizontal_arm">
         <visual>
-            <origin xyz="-0.03 -0.4 -0.06" rpy="${pi / 2.0} 0 ${pi / 2.0}" />
+            <origin xyz="-0.003 -0.04 -0.006" rpy="${pi / 2.0} 0 ${pi / 2.0}" />
             <geometry>
                 <mesh filename="package://arduinobot_description/meshes/horizontal_arm.STL"
-                    scale="0.01 0.01 0.01" />
+                    scale="0.001 0.001 0.001" />
                 <material name="grey" />
             </geometry>
@@ -77,66 +77,66 @@
         </visual>
         <collision>
-            <origin xyz="-0.03 -0.4 -0.06" rpy="${pi / 2.0} 0 ${pi / 2.0}" />
+            <origin xyz="-0.003 -0.04 -0.006" rpy="${pi / 2.0} 0 ${pi / 2.0}" />
             <geometry>
                 <mesh filename="package://arduinobot_description/meshes/horizontal_arm.STL"
-                    scale="0.01 0.01 0.01" />
+                    scale="0.001 0.001 0.001" />
                 <material name="grey" />
             </geometry>
         </collision>
-        <xacro:default_inertia mass="0.1" />
+        <xacro:default_inertia mass="0.01" />
     </link>
     <link name="claw_support">
         <visual>
-            <origin xyz="0 -0.05 -0.15" rpy="0 0 ${pi / 2.0}" />
+            <origin xyz="0 -0.005 -0.015" rpy="0 0 ${pi / 2.0}" />
             <geometry>
                 <mesh filename="package://arduinobot_description/meshes/claw_support.STL"
-                    scale="0.01 0.01 0.01" />
+                    scale="0.001 0.001 0.001" />
             </geometry>
             <material name="yellow" />
         </visual>
         <collision>
-            <origin xyz="0 -0.05 -0.15" rpy="0 0 ${pi / 2.0}" />
+            <origin xyz="0 -0.005 -0.015" rpy="0 0 ${pi / 2.0}" />
             <geometry>
                 <mesh filename="package://arduinobot_description/meshes/claw_support.STL"
-                    scale="0.01 0.01 0.01" />
+                    scale="0.001 0.001 0.001" />
             </geometry>
         </collision>
-        <xacro:default_inertia mass="0.05" />
+        <xacro:default_inertia mass="0.005" />
     </link>
     <link name="gripper_right">
         <visual>
-            <origin xyz="-0.1 0.5 -0.1" rpy="0 0 -${pi / 2.0}" />
+            <origin xyz="-0.01 0.05 -0.01" rpy="0 0 -${pi / 2.0}" />
             <geometry>
                 <mesh filename="package://arduinobot_description/meshes/right_finger.STL"
-                    scale="0.01 0.01 0.01" />
+                    scale="0.001 0.001 0.001" />
             </geometry>
             <material name="green" />
         </visual>
         <collision>
-            <origin xyz="-0.1 0.5 -0.1" rpy="0 0 -${pi / 2.0}" />
+            <origin xyz="-0.01 0.05 -0.01" rpy="0 0 -${pi / 2.0}" />
             <geometry>
                 <mesh filename="package://arduinobot_description/meshes/right_finger.STL"
-                    scale="0.01 0.01 0.01" />
+                    scale="0.001 0.001 0.001" />
             </geometry>
         </collision>
-        <xacro:default_inertia mass="0.01" />
+        <xacro:default_inertia mass="0.001" />
     </link>
     <link name="gripper_left">
         <visual>
-            <origin xyz="-0.04 0.5 -0.1" rpy="0 0 -${pi / 2.0}" />
+            <origin xyz="-0.004 0.05 -0.01" rpy="0 0 -${pi / 2.0}" />
             <geometry>
                 <mesh filename="package://arduinobot_description/meshes/left_finger.STL"
-                    scale="0.01 0.01 0.01" />
+                    scale="0.001 0.001 0.001" />
             </geometry>
             <material name="green" />
         </visual>
         <collision>
-            <origin xyz="-0.1 0.5 -0.1" rpy="0 0 -${pi / 2.0}" />
+            <origin xyz="-0.004 0.05 -0.01" rpy="0 0 -${pi / 2.0}" />
             <geometry>
-                <mesh filename="package://arduinobot_description/meshes/right_finger.STL"
-                    scale="0.01 0.01 0.01" />
+                <mesh filename="package://arduinobot_description/meshes/left_finger.STL"
+                    scale="0.001 0.001 0.001" />
             </geometry>
         </collision>
-        <xacro:default_inertia mass="0.01" />
+        <xacro:default_inertia mass="0.001" />
     </link>
     <joint name="virtual_joint" type="fixed">
@@ -146,5 +146,5 @@
     </joint>
     <joint name="joint_1" type="revolute">
-        <origin xyz="0 0 0.307" rpy="0 0 0" />
+        <origin xyz="0 0 0.0307" rpy="0 0 0" />
         <parent link="base_link" />
         <child link="base_plate" />
@@ -153,5 +153,5 @@
     </joint>
     <joint name="joint_2" type="revolute">
-        <origin xyz="-0.02 0 0.35" rpy="0 0 0" />
+        <origin xyz="-0.002 0 0.035" rpy="0 0 0" />
         <parent link="base_plate" />
         <child link="forward_drive_arm" />
@@ -160,5 +160,5 @@
     </joint>
     <joint name="joint_3" type="revolute">
-        <origin xyz="0 0 0.8" rpy="0 0 0" />
+        <origin xyz="0 0 0.08" rpy="0 0 0" />
         <parent link="forward_drive_arm" />
         <child link="horizontal_arm" />
@@ -167,10 +167,10 @@
     </joint>
     <joint name="horizontal_arm_to_claw_support" type="fixed">
-        <origin xyz="0 0.82 0" rpy="0 0 0" />
+        <origin xyz="0 0.082 0" rpy="0 0 0" />
         <parent link="horizontal_arm" />
         <child link="claw_support" />
     </joint>
     <joint name="joint_4" type="revolute">
-        <origin xyz="-0.04 0.13 -0.1" rpy="0 0 0" />
+        <origin xyz="-0.004 0.013 -0.01" rpy="0 0 0" />
         <parent link="claw_support" />
         <child link="gripper_right" />
@@ -179,5 +179,5 @@
     </joint>
     <joint name="joint_5" type="revolute">
-        <origin xyz="-0.22 0.13 -0.1" rpy="0 0 0" />
+        <origin xyz="-0.022 0.013 -0.01" rpy="0 0 0" />
         <parent link="claw_support" />
         <child link="gripper_left" />
